File: 03 Electrical/02 Schematics/ESP32-Drone/esp32.kicad_sch (KiCad schematic)
At the start: 0 parts

Commit message: started placing the esp32 circuitry
Parts:
- added U1: ESP32-C3, Package_DFN_QFN:QFN-32-1EP_5x5mm_P0.5mm_EP3.7x3.7mm, symbol MCU_Espressif:ESP32-C3
Connections:
- new net +3V3: U1.11 (VDD3P3_RTC), U1.17 (VDD3P3_CPU), U1.18 (VDD_SPI), U1.2 (VDD3P3), U1.3 (VDD3P3), U1.31 (VDDA), U1.32 (VDDA)
- new net GND_MCU: U1.33 (GND)
- new net MTCK: U1.12 (MTCK)
- new net MTDI: U1.10 (MTDI)
- new net MTDO: U1.13 (MTDO)
- new net MTMS: U1.9 (MTMS)
- no-connect marks 0 -> 1
Other:
- note added: "No antenna required for the ESP32 will be using the LoRA module to communicate with our system"
