File: 03 Electrical/02 Schematics/ESP32-Drone/ESC_motors.kicad_sch (KiCad schematic)
At the start: 0 parts

Commit message: added the two sensors for this project
Other:
- note added: "motors will be determined later on, and esc too"
Changed lines of the file:
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@@
 	(generator_version "9.0")
 	(paper "A4")
+	(text "motors will be determined later on, and esc too"
+		(exclude_from_sim no)
+		(at 100.33 67.945 0)
+		(effects
+			(font
+				(size 1.27 1.27)
+			)
+		)
+	)
 )
