File: 03 Electrical/02 Schematics/ESP32-Drone/sensors_circuit.kicad_sch (KiCad schematic)
At the start: 0 parts

Commit message: added the two sensors for this project
Parts:
- added U2: BNO055, Package_LGA:LGA-28_5.2x3.8mm_P0.5mm, symbol Sensor_Motion:BNO055
- added U3: MAX-M10S, RF_GPS:ublox_MAX, symbol RF_GPS:MAX-M10S
Connections:
- new net: U3.1 (GND), U3.10 (GND), U3.12 (GND)
Other:
- note added: "BNO055 = mag,baro,IMU,accel"
- note added: "GPS module"
Changed lines of the file:
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@@
 	(generator_version "9.0")
 	(paper "A4")
+	(text "GPS module\n"
+		(exclude_from_sim no)
+		(at 224.155 46.99 0)
+		(effects
+			(font
+				(size 1.27 1.27)
+			)
+		)
+	)
+	(text "BNO055 = mag,baro,IMU,accel\n\n"
+		(exclude_from_sim no)
+		(at 113.665 45.72 0)
+		(effects
+			(font
+				(size 1.27 1.27)
+			)
+		)
+	)
+	(symbol
+		(lib_id "RF_GPS:MAX-M10S")
+		(at 215.9 76.2 0)
+		(unit 1)
+		(exclude_from_sim no)
+		(in_bom yes)
+		(on_board yes)
+		(dnp no)
+		(fields_autoplaced yes)
+		(property "Reference" "U3"
+			(at 218.0433 93.98 0)
+			(effects
+				(font
+					(size 1.27 1.27)
+				)
+				(justify left)
+			)
+		)
+		(property "Value" "MAX-M10S"
+			(at 218.0433 96.52 0)
+			(effects
+				(font
+					(size 1.27 1.27)
+				)
+				(justify left)
+			)
+		)
+		(property "Footprint" "RF_GPS:ublox_MAX"
+			(at 226.06 92.71 0)
+			(effects
+				(font
+					(size 1.27 1.27)
+				)
+				(hide yes)
+			)
+		)
+		(property "Datasheet" "https://content.u-blox.com/sites/default/files/MAX-M10S_DataSheet_UBX-20035208.pdf"
+			(at 215.9 76.2 0)
+			(effects
+				(font
+					(size 1.27 1.27)
+				)
+				(hide yes)
+			)
+		)
+		(property "Description" "GNSS Module MAX M10, VCC 1.65V to 3.6V"
+			(at 215.9 76.2 0)
+			(effects
+				(font
+					(size 1.27 1.27)
+				)
+				(hide yes)
+			)
+		)
+		(pin "7"
+		)
+		(pin "12"
+		)
+		(pin "1"
+		)
+		(pin "9"
+		)
+		(pin "18"
+		)
+		(pin "5"
+		)
+		(pin "17"
+		)
+		(pin "16"
+		)
+		(pin "3"
+		)
+		(pin "2"
+		)
+		(pin "15"
+		)
+		(pin "6"
+		)
+		(pin "4"
+		)
+		(pin "8"
+		)
+		(pin "10"
+		)
+		(pin "14"
+		)
+		(pin "13"
+		)
+		(pin "11"
+		)
+		(instances
+			(project ""
+				(path "/2b6165e2-6038-49be-a1b7-174ab2023d42/e01dc768-0ee3-4879-b330-ecde0f6db60a"
+					(reference "U3")
+					(unit 1)
+				)
+			)
+		)
+	)
+	(symbol
+		(lib_id "Sensor_Motion:BNO055")
+		(at 113.03 73.66 0)
+		(unit 1)
+		(exclude_from_sim no)
+		(in_bom yes)
+		(on_board yes)
+		(dnp no)
+		(fields_autoplaced yes)
+		(property "Reference" "U2"
+			(at 117.7133 53.34 0)
+			(effects
+				(font
+					(size 1.27 1.27)
+				)
+				(justify left)
+			)
+		)
+		(property "Value" "BNO055"
+			(at 117.7133 55.88 0)
+			(effects
+				(font
+					(size 1.27 1.27)
+				)
+				(justify left)
+			)
+		)
+		(property "Footprint" "Package_LGA:LGA-28_5.2x3.8mm_P0.5mm"
+			(at 119.38 90.17 0)
+			(effects
+				(font
+					(size 1.27 1.27)
+				)
+				(justify left)
+				(hide yes)
+			)
+		)
+		(property "Datasheet" "https://www.bosch-sensortec.com/media/boschsensortec/downloads/datasheets/bst-bno055-ds000.pdf"
+			(at 113.03 68.58 0)
+			(effects
+				(font
+					(size 1.27 1.27)
+				)
+				(hide yes)
+			)
+		)
+		(property "Description" "Intelligent 9-axis absolute orientation sensor, LGA-28"
+			(at 113.03 73.66 0)
+			(effects
+				(font
+					(size 1.27 1.27)
+				)
+				(hide yes)
+			)
+		)
+		(pin "18"
+		)
+		(pin "19"
+		)
+		(pin "20"
+		)
+		(pin "10"
+		)
+		(pin "4"
+		)
+		(pin "14"
+		)
+		(pin "11"
+		)
+		(pin "17"
+		)
+		(pin "1"
+		)
+		(pin "7"
+		)
+		(pin "8"
+		)
+		(pin "3"
+		)
+		(pin "2"
+		)
+		(pin "28"
+		)
+		(pin "25"
+		)
+		(pin "15"
+		)
+		(pin "16"
+		)
+		(pin "12"
+		)
+		(pin "13"
+		)
+		(pin "21"
+		)
+		(pin "22"
+		)
+		(pin "23"
+		)
+		(pin "24"
+		)
+		(pin "26"
+		)
+		(pin "27"
+		)
+		(pin "6"
+		)
+		(pin "5"
+		)
+		(pin "9"
+		)
+		(instances
+			(project ""
+				(path "/2b6165e2-6038-49be-a1b7-174ab2023d42/e01dc768-0ee3-4879-b330-ecde0f6db60a"
+					(reference "U2")
+					(unit 1)
+				)
+			)
+		)
+	)
 )
