File: 03 Electrical/02 Schematics/ESP32-DRONE ANDREW/power_circuit.kicad_sch (KiCad schematic)
At the start: 0 parts

Commit message: finished power managemnt
Parts:
- added C10, C11, C14, C15, C17, C9: 1u, symbol Device:C_Small
- added C12, C13, C16, C18, C19, C20: 100n, symbol Device:C_Small
- added D2: SMAJ11CA, Diode_SMD:D_SMA, symbol Diode:SMAJ11CA
- added J1: Conn_01x02_Pin, Connector_AMASS:AMASS_XT60-F_1x02_P7.20mm_Vertical, symbol Connector:Conn_01x02_Pin
- added L1, L2, L3, L4: 4.4u, symbol Device:L_Small
- added R10: 25k, symbol Device:R_Small
- added R9: 200k, symbol Device:R_Small
- added SW1: SW_Nidec_CAS-120A1, Button_Switch_SMD:Nidec_Copal_CAS-120A, symbol Switch:SW_Nidec_CAS-120A1
- added U1: ~, Package_DFN_QFN:WDFN-8_2x2mm_P0.5mm, symbol Library 1:RT9718
- added U6, U7: LP5912-3.3DRV, Package_SON:WSON-6-1EP_2x2mm_P0.65mm_EP1x1.6mm_ThermalVias, symbol Regulator_Linear:LP5912-3.3DRV
Connections:
- new net: C14.1, L2.1, U6.1 (OUT)
- new net: C17.1, L4.1, U7.1 (OUT)
- new net: C16.1, L3.2, U7.4 (EN), U7.6 (IN)
- new net: C12.1, L1.2, U6.4 (EN), U6.6 (IN)
- new net: R9.2, U1.1 (VIN), U1.5 (EN), U1.6 (VB)
- new net: R10.1, U1.7 (ILM)
- new net +3.3V: C13.1, L2.2
- new net +3.3VA: C18.1, C19.1, C20.1, L4.2
- new net +BATT: J1.2 (Pin_2), SW1.2 (B)
- new net +VON: C9.1, D2.2 (A2), R9.1, SW1.3 (A)
- new net GND1: C10.2, C11.2, C12.2, C13.2, C14.2, C15.2, C16.2, C17.2, C18.2, C19.2, C20.2, C9.2, D2.1 (A1), J1.1 (Pin_1), R10.2, U1.2 (GND), U1.9 (GND), U6.5 (GND), U6.7 (EP), U7.5 (GND), U7.7 (EP)
- new net VCC: C10.1, C11.1, C15.1, L1.1, L3.1, U1.8 (VOUT)
- no-connect marks 0 -> 2
Other:
- note added: "CALCULATE THE OVERCURRENT PROTECTION CIRCUIT"
